Commit message: Remove dependency on pr2_description. Fixes #23.

File: urdf/05-visual.urdf (robot description, URDF)
Before this commit: robot visual, 16 links, 15 joints
Links:
- link left_gripper: geometry visual mesh filename=package://urdf_tutorial/meshes/l_finger.dae
- link left_tip: geometry visual mesh filename=package://urdf_tutorial/meshes/l_finger_tip.dae
- link right_gripper: geometry visual mesh filename=package://urdf_tutorial/meshes/l_finger.dae
- link right_tip: geometry visual mesh filename=package://urdf_tutorial/meshes/l_finger_tip.dae

File: urdf/06-flexible.urdf (robot description, URDF)
Before this commit: robot visual, 16 links, 15 joints
Links:
- link left_gripper: geometry visual mesh filename=package://urdf_tutorial/meshes/l_finger.dae
- link left_tip: geometry visual mesh filename=package://urdf_tutorial/meshes/l_finger_tip.dae
- link right_gripper: geometry visual mesh filename=package://urdf_tutorial/meshes/l_finger.dae
- link right_tip: geometry visual mesh filename=package://urdf_tutorial/meshes/l_finger_tip.dae

File: urdf/07-physics.urdf (robot description, URDF)
Before this commit: robot physics, 16 links, 15 joints
Links:
- link left_gripper: geometry collision mesh filename=package://urdf_tutorial/meshes/l_finger.dae; visual mesh filename=package://urdf_tutorial/meshes/l_finger.dae
- link left_tip: geometry collision mesh filename=package://urdf_tutorial/meshes/l_finger_tip.dae; visual mesh filename=package://urdf_tutorial/meshes/l_finger_tip.dae
- link right_gripper: geometry collision mesh filename=package://urdf_tutorial/meshes/l_finger.dae; visual mesh filename=package://urdf_tutorial/meshes/l_finger.dae
- link right_tip: geometry collision mesh filename=package://urdf_tutorial/meshes/l_finger_tip.dae; visual mesh filename=package://urdf_tutorial/meshes/l_finger_tip.dae

File: urdf/08-macroed.urdf.xacro (robot description, xacro)
@@ -140,10 +140,10 @@
         <origin rpy="${(reflect-1)/2*pi} 0 0" xyz="0 0 0"/>
         <geometry>
-          <mesh filename="package://pr2_description/meshes/gripper_v0/l_finger.dae"/>
-        </geometry>
-      </visual>
-      <collision>
-        <geometry>
-          <mesh filename="package://pr2_description/meshes/gripper_v0/l_finger.dae"/>
+          <mesh filename="package://urdf_tutorial/meshes/l_finger.dae"/>
+        </geometry>
+      </visual>
+      <collision>
+        <geometry>
+          <mesh filename="package://urdf_tutorial/meshes/l_finger.dae"/>
         </geometry>
         <origin rpy="${(reflect-1)/2*pi} 0 0" xyz="0 0 0"/>
@@ -159,10 +159,10 @@
         <origin rpy="${(reflect-1)/2*pi} 0 0" xyz="0.09137 0.00495 0"/>
         <geometry>
-          <mesh filename="package://pr2_description/meshes/gripper_v0/l_finger_tip.dae"/>
-        </geometry>
-      </visual>
-      <collision>
-        <geometry>
-          <mesh filename="package://pr2_description/meshes/gripper_v0/l_finger_tip.dae"/>
+          <mesh filename="package://urdf_tutorial/meshes/l_finger_tip.dae"/>
+        </geometry>
+      </visual>
+      <collision>
+        <geometry>
+          <mesh filename="package://urdf_tutorial/meshes/l_finger_tip.dae"/>
         </geometry>
         <origin rpy="${(reflect-1)/2*pi} 0 0" xyz="0.09137 0.00495 0"/>

File: urdf/09-roscontrol.urdf.xacro (robot description, xacro)
@@ -175,10 +175,10 @@
         <origin rpy="${(reflect-1)/2*pi} 0 0" xyz="0 0 0"/>
         <geometry>
-          <mesh filename="package://pr2_description/meshes/gripper_v0/l_finger.dae"/>
-        </geometry>
-      </visual>
-      <collision>
-        <geometry>
-          <mesh filename="package://pr2_description/meshes/gripper_v0/l_finger.dae"/>
+          <mesh filename="package://urdf_tutorial/meshes/l_finger.dae"/>
+        </geometry>
+      </visual>
+      <collision>
+        <geometry>
+          <mesh filename="package://urdf_tutorial/meshes/l_finger.dae"/>
         </geometry>
         <origin rpy="${(reflect-1)/2*pi} 0 0" xyz="0 0 0"/>
@@ -203,10 +203,10 @@
         <origin rpy="${(reflect-1)/2*pi} 0 0" xyz="0.09137 0.00495 0"/>
         <geometry>
-          <mesh filename="package://pr2_description/meshes/gripper_v0/l_finger_tip.dae"/>
-        </geometry>
-      </visual>
-      <collision>
-        <geometry>
-          <mesh filename="package://pr2_description/meshes/gripper_v0/l_finger_tip.dae"/>
+          <mesh filename="package://urdf_tutorial/meshes/l_finger_tip.dae"/>
+        </geometry>
+      </visual>
+      <collision>
+        <geometry>
+          <mesh filename="package://urdf_tutorial/meshes/l_finger_tip.dae"/>
         </geometry>
         <origin rpy="${(reflect-1)/2*pi} 0 0" xyz="0.09137 0.00495 0"/>

File: urdf/r2d2.xacro (robot description, xacro)
@@ -175,10 +175,10 @@
         <origin rpy="${(reflect-1)/2*pi} 0 0" xyz="0 0 0"/>
         <geometry>
-          <mesh filename="package://pr2_description/meshes/gripper_v0/l_finger.dae"/>
-        </geometry>
-      </visual>
-      <collision>
-        <geometry>
-          <mesh filename="package://pr2_description/meshes/gripper_v0/l_finger.dae"/>
+          <mesh filename="package://urdf_tutorial/meshes/l_finger.dae"/>
+        </geometry>
+      </visual>
+      <collision>
+        <geometry>
+          <mesh filename="package://urdf_tutorial/meshes/l_finger.dae"/>
         </geometry>
         <origin rpy="${(reflect-1)/2*pi} 0 0" xyz="0 0 0"/>
@@ -203,10 +203,10 @@
         <origin rpy="${(reflect-1)/2*pi} 0 0" xyz="0.09137 0.00495 0"/>
         <geometry>
-          <mesh filename="package://pr2_description/meshes/gripper_v0/l_finger_tip.dae"/>
-        </geometry>
-      </visual>
-      <collision>
-        <geometry>
-          <mesh filename="package://pr2_description/meshes/gripper_v0/l_finger_tip.dae"/>
+          <mesh filename="package://urdf_tutorial/meshes/l_finger_tip.dae"/>
+        </geometry>
+      </visual>
+      <collision>
+        <geometry>
+          <mesh filename="package://urdf_tutorial/meshes/l_finger_tip.dae"/>
         </geometry>
         <origin rpy="${(reflect-1)/2*pi} 0 0" xyz="0.09137 0.00495 0"/>

Commit message: Remove extra elements from static visual model

File: urdf/05-visual.urdf (robot description, URDF)
Before this commit: robot visual, 16 links, 15 joints
Joints:
- joint gripper_extension: limit lower=-0.38 upper=0 effort=1000.0 velocity=0.5 -> (none); type prismatic -> fixed
- joint left_back_wheel_joint: axis 0 1 0 -> (none)
- joint right_back_wheel_joint: axis 0 1 0 -> (none)
- joint right_front_wheel_joint: axis 0 1 0 -> (none)
