Commit message: Leading zeros

File: urdf/02-multipleshapes.urdf (robot description, URDF)
Before this commit: robot multipleshapes, 2 links, 1 joints
Links:
- link right_leg: geometry visual box size=0.6 0.1 0.2

File: urdf/03-origins.urdf (robot description, URDF)
Before this commit: robot origins, 2 links, 1 joints
Links:
- link right_leg: geometry visual box size=0.6 0.1 0.2
Joints:
- joint base_to_right_leg: origin xyz=0 -0.22 .25 -> xyz=0 -0.22 0.25

File: urdf/04-materials.urdf (robot description, URDF)
Before this commit: robot materials, 3 links, 2 joints
Links:
- link left_leg: geometry visual box size=0.6 0.1 0.2
- link right_leg: geometry visual box size=0.6 0.1 0.2
Joints:
- joint base_to_left_leg: origin xyz=0 0.22 .25 -> xyz=0 0.22 0.25
- joint base_to_right_leg: origin xyz=0 -0.22 .25 -> xyz=0 -0.22 0.25

File: urdf/05-visual.urdf (robot description, URDF)
Before this commit: robot visual, 16 links, 15 joints
Links:
- link box: geometry visual box size=0.08 0.08 0.08
- link gripper_pole: geometry visual cylinder length=0.2 radius=0.01
- link left_base: geometry visual box size=0.4 0.1 0.1
- link left_leg: geometry visual box size=0.6 0.1 0.2
- link right_base: geometry visual box size=0.4 0.1 0.1
- link right_leg: geometry visual box size=0.6 0.1 0.2
Joints:
- joint base_to_left_leg: origin xyz=0 0.22 .25 -> xyz=0 0.22 0.25
- joint base_to_right_leg: origin xyz=0 -0.22 .25 -> xyz=0 -0.22 0.25
- joint gripper_extension: origin xyz=0.19 0 .2 rpy=0 0 0 -> xyz=0.19 0 0.2 rpy=0 0 0

File: urdf/06-flexible.urdf (robot description, URDF)
Before this commit: robot visual, 16 links, 15 joints
Links:
- link box: geometry visual box size=0.08 0.08 0.08
- link gripper_pole: geometry visual cylinder length=0.2 radius=0.01
- link left_base: geometry visual box size=0.4 0.1 0.1
- link left_leg: geometry visual box size=0.6 0.1 0.2
- link right_base: geometry visual box size=0.4 0.1 0.1
- link right_leg: geometry visual box size=0.6 0.1 0.2
Joints:
- joint base_to_left_leg: origin xyz=0 0.22 .25 -> xyz=0 0.22 0.25
- joint base_to_right_leg: origin xyz=0 -0.22 .25 -> xyz=0 -0.22 0.25
- joint gripper_extension: origin xyz=0.19 0 .2 rpy=0 0 0 -> xyz=0.19 0 0.2 rpy=0 0 0

File: urdf/07-physics.urdf (robot description, URDF)
Before this commit: robot physics, 16 links, 15 joints
Links:
- link box: geometry collision box size=0.08 0.08 0.08; visual box size=0.08 0.08 0.08
- link gripper_pole: geometry collision cylinder length=0.2 radius=0.01; visual cylinder length=0.2 radius=0.01
- link left_base: geometry collision box size=0.4 0.1 0.1; visual box size=0.4 0.1 0.1
- link left_leg: geometry collision box size=0.6 0.1 0.2; visual box size=0.6 0.1 0.2
- link right_base: geometry collision box size=0.4 0.1 0.1; visual box size=0.4 0.1 0.1
- link right_leg: geometry collision box size=0.6 0.1 0.2; visual box size=0.6 0.1 0.2
Joints:
- joint base_to_left_leg: origin xyz=0 0.22 .25 -> xyz=0 0.22 0.25
- joint base_to_right_leg: origin xyz=0 -0.22 .25 -> xyz=0 -0.22 0.25
- joint gripper_extension: origin xyz=0.19 0 .2 rpy=0 0 0 -> xyz=0.19 0 0.2 rpy=0 0 0

File: urdf/08-macroed.urdf.xacro (robot description, xacro)
@@ -1,13 +1,13 @@
 <?xml version="1.0"?>
 <robot name="macroed" xmlns:xacro="http://ros.org/wiki/xacro">
-  <xacro:property name="width" value=".2" />
-  <xacro:property name="leglen" value=".6" />
-  <xacro:property name="polelen" value=".2" />
-  <xacro:property name="bodylen" value=".6" />
-  <xacro:property name="baselen" value=".4" />
-  <xacro:property name="wheeldiam" value=".07" />
+  <xacro:property name="width" value="0.2" />
+  <xacro:property name="leglen" value="0.6" />
+  <xacro:property name="polelen" value="0.2" />
+  <xacro:property name="bodylen" value="0.6" />
+  <xacro:property name="baselen" value="0.4" />
+  <xacro:property name="wheeldiam" value="0.07" />
   <xacro:property name="pi" value="3.1415" />
   <material name="blue">
-    <color rgba="0 0 .8 1"/>
+    <color rgba="0 0 0.8 1"/>
   </material>
   <material name="black">
@@ -65,5 +65,5 @@
       <visual>
         <geometry>
-          <box size="${leglen} .1 .2"/>
+          <box size="${leglen} 0.1 0.2"/>
         </geometry>
         <origin xyz="0 0 -${leglen/2}" rpy="0 ${pi/2} 0"/>
@@ -72,5 +72,5 @@
       <collision>
         <geometry>
-          <box size="${leglen} .1 .2"/>
+          <box size="${leglen} 0.1 0.2"/>
         </geometry>
         <origin xyz="0 0 -${leglen/2}" rpy="0 ${pi/2} 0"/>
@@ -81,10 +81,10 @@
       <parent link="base_link"/>
       <child link="${prefix}_leg"/>
-      <origin xyz="0 ${reflect*(width+.02)} .25" />
+      <origin xyz="0 ${reflect*(width+.02)} 0.25" />
     </joint>
     <link name="${prefix}_base">
       <visual>
         <geometry>
-          <box size="${baselen} .1 .1"/>
+          <box size="${baselen} 0.1 0.1"/>
         </geometry>
         <material name="white"/>
@@ -92,5 +92,5 @@
       <collision>
         <geometry>
-          <box size="${baselen} .1 .1"/>
+          <box size="${baselen} 0.1 0.1"/>
         </geometry>
       </collision>
@@ -111,10 +111,10 @@
     <child link="gripper_pole"/>
     <limit effort="1000.0" lower="-${width*2-.02}" upper="0" velocity="0.5"/>
-    <origin rpy="0 0 0" xyz="${width-.01} 0 .2"/>
+    <origin rpy="0 0 0" xyz="${width-.01} 0 0.2"/>
   </joint>
   <link name="gripper_pole">
     <visual>
       <geometry>
-        <cylinder length="${polelen}" radius=".01"/>
+        <cylinder length="${polelen}" radius="0.01"/>
       </geometry>
       <origin xyz="${polelen/2} 0 0" rpy="0 ${pi/2} 0 "/>
@@ -122,9 +122,9 @@
     <collision>
       <geometry>
-        <cylinder length="${polelen}" radius=".01"/>
+        <cylinder length="${polelen}" radius="0.01"/>
       </geometry>
       <origin xyz="${polelen/2} 0 0" rpy="0 ${pi/2} 0 "/>
     </collision>
-    <xacro:default_inertial mass=".05"/>
+    <xacro:default_inertial mass="0.05"/>
   </link>
   <xacro:macro name="gripper" params="prefix reflect">
@@ -149,5 +149,5 @@
         <origin rpy="${(reflect-1)/2*pi} 0 0" xyz="0 0 0"/>
       </collision>
-      <xacro:default_inertial mass=".05"/>
+      <xacro:default_inertial mass="0.05"/>
     </link>
     <joint name="${prefix}_tip_joint" type="fixed">
@@ -168,5 +168,5 @@
         <origin rpy="${(reflect-1)/2*pi} 0 0" xyz="0.09137 0.00495 0"/>
       </collision>
-      <xacro:default_inertial mass=".05"/>
+      <xacro:default_inertial mass="0.05"/>
     </link>
   </xacro:macro>
@@ -196,5 +196,5 @@
     <visual>
       <geometry>
-        <box size=".08 .08 .08"/>
+        <box size="0.08 0.08 0.08"/>
       </geometry>
       <material name="blue"/>
@@ -203,5 +203,5 @@
     <collision>
       <geometry>
-        <box size=".08 .08 .08"/>
+        <box size="0.08 0.08 0.08"/>
       </geometry>
     </collision>

File: urdf/09-roscontrol.urdf.xacro (robot description, xacro)
@@ -1,13 +1,13 @@
 <?xml version="1.0"?>
 <robot name="roscontrol" xmlns:xacro="http://ros.org/wiki/xacro">
-  <xacro:property name="width" value=".2" />
-  <xacro:property name="leglen" value=".6" />
-  <xacro:property name="polelen" value=".2" />
-  <xacro:property name="bodylen" value=".6" />
-  <xacro:property name="baselen" value=".4" />
-  <xacro:property name="wheeldiam" value=".07" />
+  <xacro:property name="width" value="0.2" />
+  <xacro:property name="leglen" value="0.6" />
+  <xacro:property name="polelen" value="0.2" />
+  <xacro:property name="bodylen" value="0.6" />
+  <xacro:property name="baselen" value="0.4" />
+  <xacro:property name="wheeldiam" value="0.07" />
   <xacro:property name="pi" value="3.1415" />
   <material name="blue">
-    <color rgba="0 0 .8 1"/>
+    <color rgba="0 0 0.8 1"/>
   </material>
   <material name="black">
@@ -87,5 +87,5 @@
       <visual>
         <geometry>
-          <box size="${leglen} .1 .2"/>
+          <box size="${leglen} 0.1 0.2"/>
         </geometry>
         <origin xyz="0 0 -${leglen/2}" rpy="0 ${pi/2} 0"/>
@@ -94,5 +94,5 @@
       <collision>
         <geometry>
-          <box size="${leglen} .1 .2"/>
+          <box size="${leglen} 0.1 0.2"/>
         </geometry>
         <origin xyz="0 0 -${leglen/2}" rpy="0 ${pi/2} 0"/>
@@ -103,10 +103,10 @@
       <parent link="base_link"/>
       <child link="${prefix}_leg"/>
-      <origin xyz="0 ${reflect*(width+.02)} .25" />
+      <origin xyz="0 ${reflect*(width+.02)} 0.25" />
     </joint>
     <link name="${prefix}_base">
       <visual>
         <geometry>
-          <box size="${baselen} .1 .1"/>
+          <box size="${baselen} 0.1 0.1"/>
         </geometry>
         <material name="white"/>
@@ -114,5 +114,5 @@
       <collision>
         <geometry>
-          <box size="${baselen} .1 .1"/>
+          <box size="${baselen} 0.1 0.1"/>
         </geometry>
       </collision>
@@ -133,5 +133,5 @@
     <child link="gripper_pole"/>
     <limit effort="1000.0" lower="-${width*2-.02}" upper="0" velocity="0.5"/>
-    <origin rpy="0 0 0" xyz="${width-.01} 0 .2"/>
+    <origin rpy="0 0 0" xyz="${width-.01} 0 0.2"/>
     <limit effort="30" velocity="0.2"/>
     <dynamics damping="0.0" friction="0.0"/>
@@ -140,5 +140,5 @@
     <visual>
       <geometry>
-        <cylinder length="${polelen}" radius=".01"/>
+        <cylinder length="${polelen}" radius="0.01"/>
       </geometry>
       <origin xyz="${polelen/2} 0 0" rpy="0 ${pi/2} 0 "/>
@@ -146,9 +146,9 @@
     <collision>
       <geometry>
-        <cylinder length="${polelen}" radius=".01"/>
+        <cylinder length="${polelen}" radius="0.01"/>
       </geometry>
       <origin xyz="${polelen/2} 0 0" rpy="0 ${pi/2} 0 "/>
     </collision>
-    <xacro:default_inertial mass=".05"/>
+    <xacro:default_inertial mass="0.05"/>
   </link>
   <transmission name="gripper_extension_trans" type="SimpleTransmission">
@@ -184,5 +184,5 @@
         <origin rpy="${(reflect-1)/2*pi} 0 0" xyz="0 0 0"/>
       </collision>
-      <xacro:default_inertial mass=".05"/>
+      <xacro:default_inertial mass="0.05"/>
     </link>
     <transmission name="${prefix}_gripper_trans" type="SimpleTransmission">
@@ -212,5 +212,5 @@
         <origin rpy="${(reflect-1)/2*pi} 0 0" xyz="0.09137 0.00495 0"/>
       </collision>
-      <xacro:default_inertial mass=".05"/>
+      <xacro:default_inertial mass="0.05"/>
     </link>
   </xacro:macro>
@@ -253,5 +253,5 @@
     <visual>
       <geometry>
-        <box size=".08 .08 .08"/>
+        <box size="0.08 0.08 0.08"/>
       </geometry>
       <material name="blue"/>
@@ -260,5 +260,5 @@
     <collision>
       <geometry>
-        <box size=".08 .08 .08"/>
+        <box size="0.08 0.08 0.08"/>
       </geometry>
     </collision>

File: urdf/r2d2.xacro (robot description, xacro)
@@ -1,13 +1,13 @@
 <?xml version="1.0"?>
 <robot name="r2d2" xmlns:xacro="http://ros.org/wiki/xacro">
-  <xacro:property name="width" value=".2" />
-  <xacro:property name="leglen" value=".6" />
-  <xacro:property name="polelen" value=".2" />
-  <xacro:property name="bodylen" value=".6" />
-  <xacro:property name="baselen" value=".4" />
-  <xacro:property name="wheeldiam" value=".07" />
+  <xacro:property name="width" value="0.2" />
+  <xacro:property name="leglen" value="0.6" />
+  <xacro:property name="polelen" value="0.2" />
+  <xacro:property name="bodylen" value="0.6" />
+  <xacro:property name="baselen" value="0.4" />
+  <xacro:property name="wheeldiam" value="0.07" />
   <xacro:property name="pi" value="3.1415" />
   <material name="blue">
-    <color rgba="0 0 .8 1"/>
+    <color rgba="0 0 0.8 1"/>
   </material>
   <material name="black">
@@ -87,5 +87,5 @@
       <visual>
         <geometry>
-          <box size="${leglen} .1 .2"/>
+          <box size="${leglen} 0.1 0.2"/>
         </geometry>
         <origin xyz="0 0 -${leglen/2}" rpy="0 ${pi/2} 0"/>
@@ -94,5 +94,5 @@
       <collision>
         <geometry>
-          <box size="${leglen} .1 .2"/>
+          <box size="${leglen} 0.1 0.2"/>
         </geometry>
         <origin xyz="0 0 -${leglen/2}" rpy="0 ${pi/2} 0"/>
@@ -103,10 +103,10 @@
       <parent link="base_link"/>
       <child link="${prefix}_leg"/>
-      <origin xyz="0 ${reflect*(width+.02)} .25" />
+      <origin xyz="0 ${reflect*(width+.02)} 0.25" />
     </joint>
     <link name="${prefix}_base">
       <visual>
         <geometry>
-          <box size="${baselen} .1 .1"/>
+          <box size="${baselen} 0.1 0.1"/>
         </geometry>
         <material name="white"/>
@@ -114,5 +114,5 @@
       <collision>
         <geometry>
-          <box size="${baselen} .1 .1"/>
+          <box size="${baselen} 0.1 0.1"/>
         </geometry>
       </collision>
@@ -133,5 +133,5 @@
     <child link="gripper_pole"/>
     <limit effort="1000.0" lower="-${width*2-.02}" upper="0" velocity="0.5"/>
-    <origin rpy="0 0 0" xyz="${width-.01} 0 .2"/>
+    <origin rpy="0 0 0" xyz="${width-.01} 0 0.2"/>
     <limit effort="30" velocity="0.2"/>
     <dynamics damping="0.0" friction="0.0"/>
@@ -140,5 +140,5 @@
     <visual>
       <geometry>
-        <cylinder length="${polelen}" radius=".01"/>
+        <cylinder length="${polelen}" radius="0.01"/>
       </geometry>
       <origin xyz="${polelen/2} 0 0" rpy="0 ${pi/2} 0 "/>
@@ -146,9 +146,9 @@
     <collision>
       <geometry>
-        <cylinder length="${polelen}" radius=".01"/>
+        <cylinder length="${polelen}" radius="0.01"/>
       </geometry>
       <origin xyz="${polelen/2} 0 0" rpy="0 ${pi/2} 0 "/>
     </collision>
-    <xacro:default_inertial mass=".05"/>
+    <xacro:default_inertial mass="0.05"/>
   </link>
   <transmission name="gripper_extension_trans" type="SimpleTransmission">
@@ -184,5 +184,5 @@
         <origin rpy="${(reflect-1)/2*pi} 0 0" xyz="0 0 0"/>
       </collision>
-      <xacro:default_inertial mass=".05"/>
+      <xacro:default_inertial mass="0.05"/>
     </link>
     <transmission name="${prefix}_gripper_trans" type="SimpleTransmission">
@@ -212,5 +212,5 @@
         <origin rpy="${(reflect-1)/2*pi} 0 0" xyz="0.09137 0.00495 0"/>
       </collision>
-      <xacro:default_inertial mass=".05"/>
+      <xacro:default_inertial mass="0.05"/>
     </link>
   </xacro:macro>
@@ -253,5 +253,5 @@
     <visual>
       <geometry>
-        <box size=".08 .08 .08"/>
+        <box size="0.08 0.08 0.08"/>
       </geometry>
       <material name="blue"/>
@@ -260,5 +260,5 @@
     <collision>
       <geometry>
-        <box size=".08 .08 .08"/>
+        <box size="0.08 0.08 0.08"/>
       </geometry>
     </collision>
