Commit message: Update final r2d2.xacro implementation with roscontrol version

File: urdf/09-roscontrol.urdf.xacro (robot description, xacro)
@@ -1,4 +1,4 @@
 <?xml version="1.0"?>
-<robot name="macroed" xmlns:xacro="http://ros.org/wiki/xacro">
+<robot name="roscontrol" xmlns:xacro="http://ros.org/wiki/xacro">
   <xacro:property name="width" value=".2" />
   <xacro:property name="leglen" value=".6" />

File: urdf/r2d2.xacro (robot description, xacro)
@@ -8,4 +8,13 @@
   <xacro:property name="wheeldiam" value=".07" />
   <xacro:property name="pi" value="3.1415" />
+  <material name="blue">
+    <color rgba="0 0 .8 1"/>
+  </material>
+  <material name="black">
+    <color rgba="0 0 0 1"/>
+  </material>
+  <material name="white">
+    <color rgba="1 1 1 1"/>
+  </material>
   <xacro:macro name="default_inertial" params="mass">
     <inertial>
@@ -19,7 +28,5 @@
         <cylinder radius="${width}" length="${bodylen}"/>
       </geometry>
-      <material name="blue">
-        <color rgba="0 0 .8 1"/>
-      </material>
+      <material name="blue"/>
     </visual>
     <collision>
@@ -33,33 +40,46 @@
     <link name="${prefix}_${suffix}_wheel">
       <visual>
-        <geometry>
-          <cylinder radius="${wheeldiam/2}" length=".1"/>
-        </geometry>
-        <material name="black">
-          <color rgba="0 0 0 1"/>
-        </material>
-      </visual>
-      <collision>
-        <geometry>
-          <cylinder radius="${wheeldiam/2}" length=".1"/>
-        </geometry>
+        <origin xyz="0 0 0" rpy="${pi/2} 0 0" />
+        <geometry>
+          <cylinder radius="${wheeldiam/2}" length="0.1"/>
+        </geometry>
+        <material name="black"/>
+        <origin xyz="0 0 0" rpy="0 0 0" />
+      </visual>
+      <collision>
+        <origin xyz="0 0 0" rpy="${pi/2} 0 0" />
+        <geometry>
+          <cylinder radius="${wheeldiam/2}" length="0.1"/>
+        </geometry>
+        <origin xyz="0 0 0" rpy="0 0 0" />
       </collision>
       <xacro:default_inertial mass="1"/>
     </link>
     <joint name="${prefix}_${suffix}_wheel_joint" type="continuous">
-      <axis xyz="0 0 1"/>
+      <axis xyz="0 1 0" rpy="0 0 0" />
       <parent link="${prefix}_base"/>
       <child link="${prefix}_${suffix}_wheel"/>
-      <origin xyz="0 ${baselen*reflect/3} -${wheeldiam/2+.05}" rpy="0 ${pi/2} 0"/>
-      <limit effort="100" velocity="100" />
-      <joint_properties damping="0.0" friction="0.0" />
-    </joint>
-    <gazebo reference="${prefix}_${suffix}_wheel" >
-      <mu1>50.0</mu1>
-      <mu2>50.0</mu2>
-      <kp>100000000.0</kp>
-      <kd>1.0</kd>
-      <material>Gazebo/Fish</material>
+      <origin xyz="${baselen*reflect/3} 0 -${wheeldiam/2+.05}" rpy="0 0 0"/>
+    </joint>
+    <!-- This block provides the simulator (Gazebo) with information on a few additional
+    physical properties. See http://gazebosim.org/tutorials/?tut=ros_urdf for more-->
+    <gazebo reference="${prefix}_${suffix}_wheel">
+      <mu1 value="200.0"/>
+      <mu2 value="100.0"/>
+      <kp value="10000000.0" />
+      <kd value="1.0" />
+      <material>Gazebo/Grey</material>
     </gazebo>
+    <!-- This block connects the wheel joint to an actuator (motor), which informs both
+    simulation and visualization of the robot -->
+    <transmission name="${prefix}_${suffix}_wheel_trans" type="SimpleTransmission">
+      <type>transmission_interface/SimpleTransmission</type>
+      <actuator name="${prefix}_${suffix}_wheel_motor">
+        <mechanicalReduction>1</mechanicalReduction>
+      </actuator>
+      <joint name="${prefix}_${suffix}_wheel_joint">
+        <hardwareInterface>VelocityJointInterface</hardwareInterface>
+      </joint>
+    </transmission>
   </xacro:macro>
   <xacro:macro name="leg" params="prefix reflect">
@@ -67,14 +87,12 @@
       <visual>
         <geometry>
-          <box size="${leglen} .2 .1"/>
+          <box size="${leglen} .1 .2"/>
         </geometry>
         <origin xyz="0 0 -${leglen/2}" rpy="0 ${pi/2} 0"/>
-        <material name="white">
-          <color rgba="1 1 1 1"/>
-        </material>
-      </visual>
-      <collision>
-        <geometry>
-          <box size="${leglen} .2 .1"/>
+        <material name="white"/>
+      </visual>
+      <collision>
+        <geometry>
+          <box size="${leglen} .1 .2"/>
         </geometry>
         <origin xyz="0 0 -${leglen/2}" rpy="0 ${pi/2} 0"/>
@@ -85,10 +103,10 @@
       <parent link="base_link"/>
       <child link="${prefix}_leg"/>
-      <origin xyz="${reflect*(width+.02)} 0 .25" />
+      <origin xyz="0 ${reflect*(width+.02)} .25" />
     </joint>
     <link name="${prefix}_base">
       <visual>
         <geometry>
-          <box size=".1 ${baselen} .1"/>
+          <box size="${baselen} .1 .1"/>
         </geometry>
         <material name="white"/>
@@ -96,5 +114,5 @@
       <collision>
         <geometry>
-          <box size=".1 ${baselen} .1"/>
+          <box size="${baselen} .1 .1"/>
         </geometry>
       </collision>
@@ -109,11 +127,13 @@
     <xacro:wheel prefix="${prefix}" suffix="back" reflect="-1"/>
   </xacro:macro>
-  <xacro:leg prefix="right" reflect="1" />
-  <xacro:leg prefix="left" reflect="-1" />
+  <xacro:leg prefix="right" reflect="-1" />
+  <xacro:leg prefix="left" reflect="1" />
   <joint name="gripper_extension" type="prismatic">
     <parent link="base_link"/>
     <child link="gripper_pole"/>
     <limit effort="1000.0" lower="-${width*2-.02}" upper="0" velocity="0.5"/>
-    <origin rpy="0 0 ${pi/2}" xyz="0 ${width-.01} .2"/>
+    <origin rpy="0 0 0" xyz="${width-.01} 0 .2"/>
+    <limit effort="30" velocity="0.2"/>
+    <dynamics damping="0.0" friction="0.0"/>
   </joint>
   <link name="gripper_pole">
@@ -132,4 +152,13 @@
     <xacro:default_inertial mass=".05"/>
   </link>
+  <transmission name="gripper_extension_trans" type="SimpleTransmission">
+    <type>transmission_interface/SimpleTransmission</type>
+    <actuator name="gripper_extension_motor">
+      <mechanicalReduction>1</mechanicalReduction>
+    </actuator>
+    <joint name="gripper_extension">
+      <hardwareInterface>PositionJointInterface</hardwareInterface>
+    </joint>
+  </transmission>
   <xacro:macro name="gripper" params="prefix reflect">
     <joint name="${prefix}_gripper_joint" type="revolute">
@@ -139,4 +168,6 @@
       <parent link="gripper_pole"/>
       <child link="${prefix}_gripper"/>
+      <limit effort="30" velocity="1.0"/>
+      <dynamics damping="0.0" friction="0.0"/>
     </joint>
     <link name="${prefix}_gripper">
@@ -155,4 +186,13 @@
       <xacro:default_inertial mass=".05"/>
     </link>
+    <transmission name="${prefix}_gripper_trans" type="SimpleTransmission">
+      <type>transmission_interface/SimpleTransmission</type>
+      <actuator name="${prefix}_gripper_motor">
+        <mechanicalReduction>1</mechanicalReduction>
+      </actuator>
+      <joint name="${prefix}_gripper_joint">
+        <hardwareInterface>PositionJointInterface</hardwareInterface>
+      </joint>
+    </transmission>
     <joint name="${prefix}_tip_joint" type="fixed">
       <parent link="${prefix}_gripper"/>
@@ -189,5 +229,5 @@
       </geometry>
     </collision>
-    <xacro:default_inertial mass="10"/>
+    <xacro:default_inertial mass="2"/>
   </link>
   <joint name="head_swivel" type="continuous">
@@ -196,5 +236,18 @@
     <axis xyz="0 0 1"/>
     <origin xyz="0 0 ${bodylen/2}"/>
+    <limit effort="30" velocity="1.0"/>
+    <dynamics damping="0.0" friction="0.0"/>
   </joint>
+  <!-- This block connects the head_swivel joint to an actuator (motor), which informs both
+  simulation and visualization of the robot -->
+  <transmission name="head_swivel_trans" type="SimpleTransmission">
+    <type>transmission_interface/SimpleTransmission</type>
+    <actuator name="$head_swivel_motor">
+      <mechanicalReduction>1</mechanicalReduction>
+    </actuator>
+    <joint name="head_swivel">
+      <hardwareInterface>PositionJointInterface</hardwareInterface>
+    </joint>
+  </transmission>
   <link name="box">
     <visual>
@@ -203,4 +256,5 @@
       </geometry>
       <material name="blue"/>
+      <origin xyz="-0.04 0 0"/>
     </visual>
     <collision>
@@ -214,35 +268,11 @@
     <parent link="head"/>
     <child link="box"/>
-    <origin xyz="0 ${.707*width} ${.707*width}"/>
+    <origin xyz="${.707*width+0.04} 0 ${.707*width}"/>
   </joint>
+  <!-- Gazebo plugin for ROS Control -->
   <gazebo>
-    <controller:differential_position2d name="controller1">
-      <update>100</update>
-      <leftJoint>left_back_wheel_joint</leftJoint>
-      <rightJoint>right_back_wheel_joint</rightJoint>
-      <wheelSeparation>${width}</wheelSeparation>
-      <wheelDiameter>${wheeldiam}</wheelDiameter>
-      <torque>5</torque>
-      <interface:position name="position_iface_0"/>
-    </controller:differential_position2d>
-    <controller:gazebo_ros_p3d name="p3d_base_controller" plugin="libgazebo_ros_p3d.so">
-      <alwaysOn>true</alwaysOn>
-      <updateRate>100.0</updateRate>
-      <bodyName>base_link</bodyName>
-      <topicName>base_pose_ground_truth</topicName>
-      <gaussianNoise>0.01</gaussianNoise>
-      <frameName>map</frameName>
-      <xyzOffsets>25.7 25.7 0</xyzOffsets> <!-- initialize odometry for fake localization-->
-      <rpyOffsets>0 0 0</rpyOffsets>
-      <interface:position name="p3d_base_position"/>
-    </controller:gazebo_ros_p3d>
-    <!-- this publishes empty joint_states due to no transmission, but
-    triggering robot_state_puublisher to publish tf between fixed joints in erratic,
-    (e.g. base_laser_link for the base_scan frame) -->
-    <controller:gazebo_ros_controller_manager name="gazebo_ros_controller_manager" plugin="libgazebo_ros_controller_manager.so">
-      <alwaysOn>true</alwaysOn>
-      <updateRate>1000.0</updateRate>
-      <interface:audio name="gazebo_ros_controller_manager_dummy_iface" />
-    </controller:gazebo_ros_controller_manager>
+    <plugin name="gazebo_ros_control" filename="libgazebo_ros_control.so">
+      <robotNamespace>/</robotNamespace>
+    </plugin>
   </gazebo>
 </robot>

Commit message: More cleanup

File: urdf/09-roscontrol.urdf.xacro (robot description, xacro)
@@ -45,5 +45,4 @@
         </geometry>
         <material name="black"/>
-        <origin xyz="0 0 0" rpy="0 0 0" />
       </visual>
       <collision>
@@ -52,5 +51,4 @@
           <cylinder radius="${wheeldiam/2}" length="0.1"/>
         </geometry>
-        <origin xyz="0 0 0" rpy="0 0 0" />
       </collision>
       <xacro:default_inertial mass="1"/>
@@ -73,5 +71,5 @@
     <!-- This block connects the wheel joint to an actuator (motor), which informs both
     simulation and visualization of the robot -->
-    <transmission name="${prefix}_${suffix}_wheel_trans" type="SimpleTransmission">
+    <transmission name="${prefix}_${suffix}_wheel_trans">
       <type>transmission_interface/SimpleTransmission</type>
       <actuator name="${prefix}_${suffix}_wheel_motor">
@@ -152,5 +150,5 @@
     <xacro:default_inertial mass="0.05"/>
   </link>
-  <transmission name="gripper_extension_trans" type="SimpleTransmission">
+  <transmission name="gripper_extension_trans">
     <type>transmission_interface/SimpleTransmission</type>
     <actuator name="gripper_extension_motor">
@@ -186,5 +184,5 @@
       <xacro:default_inertial mass="0.05"/>
     </link>
-    <transmission name="${prefix}_gripper_trans" type="SimpleTransmission">
+    <transmission name="${prefix}_gripper_trans">
       <type>transmission_interface/SimpleTransmission</type>
       <actuator name="${prefix}_gripper_motor">
@@ -241,5 +239,5 @@
   <!-- This block connects the head_swivel joint to an actuator (motor), which informs both
   simulation and visualization of the robot -->
-  <transmission name="head_swivel_trans" type="SimpleTransmission">
+  <transmission name="head_swivel_trans">
     <type>transmission_interface/SimpleTransmission</type>
     <actuator name="$head_swivel_motor">

File: urdf/r2d2.xacro (robot description, xacro)
@@ -45,5 +45,4 @@
         </geometry>
         <material name="black"/>
-        <origin xyz="0 0 0" rpy="0 0 0" />
       </visual>
       <collision>
@@ -52,5 +51,4 @@
           <cylinder radius="${wheeldiam/2}" length="0.1"/>
         </geometry>
-        <origin xyz="0 0 0" rpy="0 0 0" />
       </collision>
       <xacro:default_inertial mass="1"/>
@@ -73,5 +71,5 @@
     <!-- This block connects the wheel joint to an actuator (motor), which informs both
     simulation and visualization of the robot -->
-    <transmission name="${prefix}_${suffix}_wheel_trans" type="SimpleTransmission">
+    <transmission name="${prefix}_${suffix}_wheel_trans">
       <type>transmission_interface/SimpleTransmission</type>
       <actuator name="${prefix}_${suffix}_wheel_motor">
@@ -152,5 +150,5 @@
     <xacro:default_inertial mass="0.05"/>
   </link>
-  <transmission name="gripper_extension_trans" type="SimpleTransmission">
+  <transmission name="gripper_extension_trans">
     <type>transmission_interface/SimpleTransmission</type>
     <actuator name="gripper_extension_motor">
@@ -186,5 +184,5 @@
       <xacro:default_inertial mass="0.05"/>
     </link>
-    <transmission name="${prefix}_gripper_trans" type="SimpleTransmission">
+    <transmission name="${prefix}_gripper_trans">
       <type>transmission_interface/SimpleTransmission</type>
       <actuator name="${prefix}_gripper_motor">
@@ -241,5 +239,5 @@
   <!-- This block connects the head_swivel joint to an actuator (motor), which informs both
   simulation and visualization of the robot -->
-  <transmission name="head_swivel_trans" type="SimpleTransmission">
+  <transmission name="head_swivel_trans">
     <type>transmission_interface/SimpleTransmission</type>
     <actuator name="$head_swivel_motor">
