Commit message: Closes #22

File: urdf/08-macroed.urdf.xacro (robot description, xacro)
@@ -45,5 +45,4 @@
         </geometry>
         <material name="black"/>
-        <origin xyz="0 0 0" rpy="0 0 0" />
       </visual>
       <collision>
@@ -52,5 +51,4 @@
           <cylinder radius="${wheeldiam/2}" length="0.1"/>
         </geometry>
-        <origin xyz="0 0 0" rpy="0 0 0" />
       </collision>
       <xacro:default_inertial mass="1"/>

Commit message: feat: Port over urdf_tutorial to foxy

File: urdf/08-macroed.urdf.xacro (robot description, xacro)
@@ -7,5 +7,4 @@
   <xacro:property name="baselen" value="0.4" />
   <xacro:property name="wheeldiam" value="0.07" />
-  <xacro:property name="pi" value="3.1415" />
   <material name="blue">
     <color rgba="0 0 0.8 1"/>

Commit message: More reasonable inertia values.
To cite the URDF tutorial on physical properties (http://docs.ros.org/en/galactic/Tutorials/URDF/Adding-Physical-and-Collision-Properties-to-a-URDF-Model.html):
"If unsure what to put, a matrix with ixx/iyy/izz=1e-3 or smaller is often a reasonable default for a mid-sized link (it corresponds to a box of 0.1 m side length with a mass of 0.6 kg). The identity matrix is a particularly bad choice, since it is often much too high (it corresponds to a box of 0.1 m side length with a mass of 600 kg!)."
For pedagogic reasons, the urdf_tutorial examples should not do the opposite of this.

File: urdf/08-macroed.urdf.xacro (robot description, xacro)
@@ -19,5 +19,5 @@
     <inertial>
       <mass value="${mass}" />
-      <inertia ixx="1.0" ixy="0.0" ixz="0.0" iyy="1.0" iyz="0.0" izz="1.0" />
+      <inertia ixx="1e-3" ixy="0.0" ixz="0.0" iyy="1e-3" iyz="0.0" izz="1e-3" />
     </inertial>
   </xacro:macro>
